Commit message: Added simple trans1 and ros_control plugin to urdf file

File: arm_description/urdf/arm.xacro (robot description, xacro)
@@ -3,4 +3,10 @@
     <xacro:include filename="$(find arm_description)/urdf/constants.xacro"/>
     <xacro:include filename="$(find arm_description)/urdf/materials.xacro"/>
+	<gazebo>
+		<plugin name="gazebo_ros_control" filename="libgazebo_ros_control.so">
+	    	<robotNamespace>/MYROBOT</robotNamespace>
+	    	<robotSimType>gazebo_ros_control/DefaultRobotHWSim</robotSimType>
+	  	</plugin>
+	</gazebo>
     <link name="world"/>
     <link name="base_link">
@@ -62,4 +68,14 @@
         <limit effort="0" lower="${-DEG2RAD * 170}" upper="${DEG2RAD * 170}" velocity="${DEG2RAD * 300}"/>
     </joint>
+	<transmission name="tran1">
+        <type>transmission_interface/SimpleTransmission</type>
+        <joint name="q1">
+            <hardwareInterface>EffortJointInterface</hardwareInterface>
+        </joint>
+        <actuator name="motor1">
+            <hardwareInterface>EffortJointInterface</hardwareInterface>
+            <mechanicalReduction>1</mechanicalReduction>
+        </actuator>
+    </transmission>
     <link name="link_2">
         <visual>
