Commit message: Added controllers

File: arm_description/urdf/arm.urdf.xacro (robot description, xacro)
@@ -1,12 +1,6 @@
 <?xml version="1.0"?>
-<robot name="kuka_kr10r1100sixx" xmlns:xacro="http://wiki.ros.org/xacro">
+<robot name="kuka_arm" xmlns:xacro="http://wiki.ros.org/xacro">
     <xacro:include filename="$(find arm_description)/urdf/constants.xacro"/>
     <xacro:include filename="$(find arm_description)/urdf/materials.xacro"/>
-	<gazebo>
-		<plugin name="gazebo_ros_control" filename="libgazebo_ros_control.so">
-	    	<robotNamespace>/MYROBOT</robotNamespace>
-	    	<robotSimType>gazebo_ros_control/DefaultRobotHWSim</robotSimType>
-	  	</plugin>
-	</gazebo>
     <link name="world"/>
     <link name="base_link">
@@ -67,15 +61,16 @@
         <axis xyz="0 0 -1"/>
         <limit effort="0" lower="${-DEG2RAD * 170}" upper="${DEG2RAD * 170}" velocity="${DEG2RAD * 300}"/>
+	<dynamics damping="0.5"/>
     </joint>
 	<transmission name="tran1">
-        <type>transmission_interface/SimpleTransmission</type>
-        <joint name="q1">
-            <hardwareInterface>EffortJointInterface</hardwareInterface>
-        </joint>
-        <actuator name="motor1">
-            <hardwareInterface>EffortJointInterface</hardwareInterface>
-            <mechanicalReduction>1</mechanicalReduction>
-        </actuator>
-    </transmission>
+		<type>transmission_interface/SimpleTransmission</type>
+		<joint name="q1">
+			<hardwareInterface>hardware_interface/EffortJointInterface</hardwareInterface>
+		</joint>
+		<actuator name="motor1">
+			<hardwareInterface>hardware_interface/EffortJointInterface</hardwareInterface>
+			<mechanicalReduction>1</mechanicalReduction>
+		</actuator>
+	</transmission>
     <link name="link_2">
         <visual>
@@ -107,5 +102,16 @@
         <axis xyz="0 1 0"/>
         <limit effort="0" lower="${-DEG2RAD * 190}" upper="${DEG2RAD * 45}" velocity="${DEG2RAD * 225}"/>
-    </joint>
+	<dynamics damping="0.5"/>
+    </joint>
+    <transmission name="tran2">
+        <type>transmission_interface/SimpleTransmission</type>
+        <joint name="q2">
+            <hardwareInterface>hardware_interface/EffortJointInterface</hardwareInterface>
+        </joint>
+        <actuator name="motor2">
+            <hardwareInterface>hardware_interface/EffortJointInterface</hardwareInterface>
+            <mechanicalReduction>1</mechanicalReduction>
+        </actuator>
+    </transmission>
     <link name="link_3">
             <visual>
@@ -137,5 +143,16 @@
         <axis xyz="0 1 0"/>
         <limit effort="0" lower="${-DEG2RAD * 120}" upper="${DEG2RAD * 156}" velocity="${DEG2RAD * 225}"/>
-    </joint>
+	<dynamics damping="0.5"/>
+    </joint>
+	<transmission name="tran3">
+        <type>transmission_interface/SimpleTransmission</type>
+        <joint name="q3">
+            <hardwareInterface>hardware_interface/EffortJointInterface</hardwareInterface>
+        </joint>
+        <actuator name="motor3">
+            <hardwareInterface>hardware_interface/EffortJointInterface</hardwareInterface>
+            <mechanicalReduction>1</mechanicalReduction>
+        </actuator>
+    </transmission>
     <link name="link_4">
             <visual>
@@ -167,5 +184,16 @@
         <axis xyz="-1 0 0"/>
         <limit effort="0" lower="${-DEG2RAD * 185}" upper="${DEG2RAD * 185}" velocity="${DEG2RAD * 381}"/>
-    </joint>
+	<dynamics damping="0.5"/>
+    </joint>
+    <transmission name="tran4">
+        <type>transmission_interface/SimpleTransmission</type>
+        <joint name="q4">
+            <hardwareInterface>hardware_interface/EffortJointInterface</hardwareInterface>
+        </joint>
+        <actuator name="motor4">
+            <hardwareInterface>hardware_interface/EffortJointInterface</hardwareInterface>
+            <mechanicalReduction>1</mechanicalReduction>
+        </actuator>
+	</transmission>
     <link name="link_5">
             <visual>
@@ -197,5 +225,16 @@
         <axis xyz="0 1 0"/>
         <limit effort="0" lower="${-DEG2RAD * 120}" upper="${DEG2RAD * 120}" velocity="${DEG2RAD * 311}"/>
-    </joint>
+	<dynamics damping="0.5"/>
+    </joint>
+    <transmission name="tran5">
+        <type>transmission_interface/SimpleTransmission</type>
+        <joint name="q5">
+            <hardwareInterface>hardware_interface/EffortJointInterface</hardwareInterface>
+        </joint>
+        <actuator name="motor5">
+            <hardwareInterface>hardware_interface/EffortJointInterface</hardwareInterface>
+            <mechanicalReduction>1</mechanicalReduction>
+        </actuator>
+    </transmission>
     <link name="link_6">
             <visual>
@@ -227,5 +266,16 @@
         <axis xyz="-1 0 0"/>
         <limit effort="0" lower="${-DEG2RAD * 350}" upper="${DEG2RAD * 350}" velocity="${DEG2RAD * 492}"/>
-    </joint>
+	<dynamics damping="0.5"/>
+    </joint>
+    <transmission name="tran6">
+        <type>transmission_interface/SimpleTransmission</type>
+        <joint name="q6">
+            <hardwareInterface>hardware_interface/EffortJointInterface</hardwareInterface>
+        </joint>
+        <actuator name="motor6">
+            <hardwareInterface>hardware_interface/EffortJointInterface</hardwareInterface>
+            <mechanicalReduction>1</mechanicalReduction>
+        </actuator>
+    </transmission>
     <link name="tool"/>
     <joint name="link_6-tool" type="fixed">
@@ -234,3 +284,8 @@
         <origin xyz="0 0 0" rpy="0 ${DEG2RAD * 90} 0"/>
     </joint>
+	<gazebo>
+		<plugin name="gazebo_ros_control" filename="libgazebo_ros_control.so">
+			<robotNamespace>/kuka_arm</robotNamespace>
+		</plugin>
+	</gazebo>
 </robot>

Commit message: Added python script and changed launch files

File: arm_description/urdf/arm.urdf.xacro (robot description, xacro)
@@ -61,5 +61,5 @@
         <axis xyz="0 0 -1"/>
         <limit effort="0" lower="${-DEG2RAD * 170}" upper="${DEG2RAD * 170}" velocity="${DEG2RAD * 300}"/>
-	<dynamics damping="0.5"/>
+	<dynamics damping="0.0" friction="0.0"/>
     </joint>
 	<transmission name="tran1">
@@ -102,5 +102,5 @@
         <axis xyz="0 1 0"/>
         <limit effort="0" lower="${-DEG2RAD * 190}" upper="${DEG2RAD * 45}" velocity="${DEG2RAD * 225}"/>
-	<dynamics damping="0.5"/>
+	<dynamics damping="0.0" friction="0.0"/>
     </joint>
     <transmission name="tran2">
@@ -143,5 +143,5 @@
         <axis xyz="0 1 0"/>
         <limit effort="0" lower="${-DEG2RAD * 120}" upper="${DEG2RAD * 156}" velocity="${DEG2RAD * 225}"/>
-	<dynamics damping="0.5"/>
+	<dynamics damping="0.0" friction="0.0"/>
     </joint>
 	<transmission name="tran3">
@@ -184,5 +184,5 @@
         <axis xyz="-1 0 0"/>
         <limit effort="0" lower="${-DEG2RAD * 185}" upper="${DEG2RAD * 185}" velocity="${DEG2RAD * 381}"/>
-	<dynamics damping="0.5"/>
+	<dynamics damping="0.0" friction="0.0"/>
     </joint>
     <transmission name="tran4">
@@ -225,5 +225,5 @@
         <axis xyz="0 1 0"/>
         <limit effort="0" lower="${-DEG2RAD * 120}" upper="${DEG2RAD * 120}" velocity="${DEG2RAD * 311}"/>
-	<dynamics damping="0.5"/>
+	<dynamics damping="0.0" friction="0.0"/>
     </joint>
     <transmission name="tran5">
@@ -266,5 +266,5 @@
         <axis xyz="-1 0 0"/>
         <limit effort="0" lower="${-DEG2RAD * 350}" upper="${DEG2RAD * 350}" velocity="${DEG2RAD * 492}"/>
-	<dynamics damping="0.5"/>
+	<dynamics damping="0.0" friction="0.0"/>
     </joint>
     <transmission name="tran6">
@@ -287,4 +287,5 @@
 		<plugin name="gazebo_ros_control" filename="libgazebo_ros_control.so">
 			<robotNamespace>/kuka_arm</robotNamespace>
+			<robotSimType>gazebo_ros_control/DefaultRobotHWSim</robotSimType>
 		</plugin>
 	</gazebo>
