Commit message: Combined arm_sensor and arm_control. Formatted all files. Completed integration test

File: arm_description/urdf/arm.urdf.xacro (robot description, xacro)
@@ -1,106 +1,97 @@
-<?xml version="1.0"?>
+<?xml version="1.0" ?>
 <robot name="kuka_arm" xmlns:xacro="http://wiki.ros.org/xacro">
-    <xacro:include filename="$(find arm_description)/urdf/constants.xacro"/>
-    <xacro:include filename="$(find arm_description)/urdf/materials.xacro"/>
-    <link name="world"/>
+    <xacro:include filename="$(find arm_description)/urdf/constants.xacro" />
+    <xacro:include filename="$(find arm_description)/urdf/materials.xacro" />
+    <link name="world" />
     <link name="base_link">
         <visual>
-            <origin xyz="0 0 0" rpy="0 0 0"/>
-            <geometry>
-                <mesh filename="package://arm_description/meshes/visual/base_link.stl"/>
-            </geometry>
-            <xacro:material_base_frame/>
-        </visual>
-        <collision>
-            <origin xyz="0 0 0" rpy="0 0 0"/>
-            <geometry>
-                <mesh filename="package://arm_description/meshes/collision/base_link.stl"/>
-            </geometry>
-        </collision>
-        <inertial>
-            <origin xyz="0 0 0" rpy="0 0 0"/>
-            <mass value="16.8"/>
-            <inertia
-                    ixx="0.312" ixy="-0.000195" ixz="0.0809"
-                    iyy="0.411" iyz="0.0000657"
-                    izz="0.186"/>
+            <origin xyz="0 0 0" rpy="0 0 0" />
+            <geometry>
+                <mesh filename="package://arm_description/meshes/visual/base_link.stl" />
+            </geometry>
+            <xacro:material_base_frame />
+        </visual>
+        <collision>
+            <origin xyz="0 0 0" rpy="0 0 0" />
+            <geometry>
+                <mesh filename="package://arm_description/meshes/collision/base_link.stl" />
+            </geometry>
+        </collision>
+        <inertial>
+            <origin xyz="0 0 0" rpy="0 0 0" />
+            <mass value="16.8" />
+            <inertia ixx="0.312" ixy="-0.000195" ixz="0.0809" iyy="0.411" iyz="0.0000657" izz="0.186" />
         </inertial>
     </link>
     <joint name="world-base_link" type="fixed">
-            <origin xyz="0 0 0" rpy="0 0 0"/>
-            <parent link="world"/>
-            <child link="base_link"/>
+        <origin xyz="0 0 0" rpy="0 0 0" />
+        <parent link="world" />
+        <child link="base_link" />
     </joint>
     <link name="link_1">
         <visual>
-            <origin xyz="0 0 0" rpy="0 0 0"/>
-            <geometry>
-                <mesh filename="package://arm_description/meshes/visual/link_1.stl"/>
-            </geometry>
-            <xacro:material_moving_parts/>
-        </visual>
-        <collision>
-            <origin xyz="0 0 0" rpy="0 0 0"/>
-            <geometry>
-                <mesh filename="package://arm_description/meshes/collision/link_1.stl"/>
-            </geometry>
-        </collision>
-        <inertial>
-                <origin xyz="0 0 0" rpy="0 0 0"/>
-                <mass value="10.0"/>
-                <inertia
-                        ixx="1.24" ixy="-0.000146" ixz="-0.0353"
-                        iyy="1.19" iyz="-0.00761"
-                        izz="0.0912"/>
+            <origin xyz="0 0 0" rpy="0 0 0" />
+            <geometry>
+                <mesh filename="package://arm_description/meshes/visual/link_1.stl" />
+            </geometry>
+            <xacro:material_moving_parts />
+        </visual>
+        <collision>
+            <origin xyz="0 0 0" rpy="0 0 0" />
+            <geometry>
+                <mesh filename="package://arm_description/meshes/collision/link_1.stl" />
+            </geometry>
+        </collision>
+        <inertial>
+            <origin xyz="0 0 0" rpy="0 0 0" />
+            <mass value="10.0" />
+            <inertia ixx="1.24" ixy="-0.000146" ixz="-0.0353" iyy="1.19" iyz="-0.00761" izz="0.0912" />
         </inertial>
     </link>
     <joint name="q1" type="revolute">
-        <origin xyz="0 0 0.400" rpy="0 0 0"/>
-        <parent link="base_link"/>
-        <child link="link_1"/>
-        <axis xyz="0 0 -1"/>
-        <limit effort="100" lower="${-DEG2RAD * 170}" upper="${DEG2RAD * 170}" velocity="${DEG2RAD * 300}"/>
-	<dynamics damping="0.0" friction="0.0"/>
-    </joint>
-	<transmission name="tran1">
-		<type>transmission_interface/SimpleTransmission</type>
-		<joint name="q1">
-			<hardwareInterface>hardware_interface/EffortJointInterface</hardwareInterface>
-		</joint>
-		<actuator name="motor1">
-			<hardwareInterface>hardware_interface/EffortJointInterface</hardwareInterface>
-			<mechanicalReduction>1</mechanicalReduction>
-		</actuator>
-	</transmission>
+        <origin xyz="0 0 0.400" rpy="0 0 0" />
+        <parent link="base_link" />
+        <child link="link_1" />
+        <axis xyz="0 0 -1" />
+        <limit effort="100" lower="${-DEG2RAD * 170}" upper="${DEG2RAD * 170}" velocity="${DEG2RAD * 300}" />
+        <dynamics damping="0.0" friction="0.0" />
+    </joint>
+    <transmission name="tran1">
+        <type>transmission_interface/SimpleTransmission</type>
+        <joint name="q1">
+            <hardwareInterface>hardware_interface/EffortJointInterface</hardwareInterface>
+        </joint>
+        <actuator name="motor1">
+            <hardwareInterface>hardware_interface/EffortJointInterface</hardwareInterface>
+            <mechanicalReduction>1</mechanicalReduction>
+        </actuator>
+    </transmission>
     <link name="link_2">
         <visual>
-            <origin xyz="0 0 0" rpy="0 0 0"/>
-            <geometry>
-                <mesh filename="package://arm_description/meshes/visual/link_2.stl"/>
-            </geometry>
-            <xacro:material_moving_parts/>
-        </visual>
-        <collision>
-            <origin xyz="0 0 0" rpy="0 0 0"/>
-            <geometry>
-                <mesh filename="package://arm_description/meshes/collision/link_2.stl"/>
-            </geometry>
-        </collision>
-        <inertial>
-                <origin xyz="0 0 0" rpy="0 0 0"/>
-                <mass value="16.2"/>
-                <inertia
-                        ixx="7.81" ixy="0.00140" ixz="-0.176"
-                        iyy="7.78" iyz="0.0459"
-                        izz="0.0767"/>
+            <origin xyz="0 0 0" rpy="0 0 0" />
+            <geometry>
+                <mesh filename="package://arm_description/meshes/visual/link_2.stl" />
+            </geometry>
+            <xacro:material_moving_parts />
+        </visual>
+        <collision>
+            <origin xyz="0 0 0" rpy="0 0 0" />
+            <geometry>
+                <mesh filename="package://arm_description/meshes/collision/link_2.stl" />
+            </geometry>
+        </collision>
+        <inertial>
+            <origin xyz="0 0 0" rpy="0 0 0" />
+            <mass value="16.2" />
+            <inertia ixx="7.81" ixy="0.00140" ixz="-0.176" iyy="7.78" iyz="0.0459" izz="0.0767" />
         </inertial>
     </link>
     <joint name="q2" type="revolute">
-        <origin xyz="0.025 0 0" rpy="0 0 0"/>
-        <parent link="link_1"/>
-        <child link="link_2"/>
-        <axis xyz="0 1 0"/>
-        <limit effort="100" lower="${-DEG2RAD * 190}" upper="${DEG2RAD * 45}" velocity="${DEG2RAD * 225}"/>
-	<dynamics damping="0.0" friction="0.0"/>
+        <origin xyz="0.025 0 0" rpy="0 0 0" />
+        <parent link="link_1" />
+        <child link="link_2" />
+        <axis xyz="0 1 0" />
+        <limit effort="100" lower="${-DEG2RAD * 190}" upper="${DEG2RAD * 45}" velocity="${DEG2RAD * 225}" />
+        <dynamics damping="0.0" friction="0.0" />
     </joint>
     <transmission name="tran2">
@@ -115,35 +106,32 @@
     </transmission>
     <link name="link_3">
-            <visual>
-                <origin xyz="0 0 0" rpy="0 0 0"/>
-                <geometry>
-                    <mesh filename="package://arm_description/meshes/visual/link_3.stl"/>
-                </geometry>
-                <xacro:material_moving_parts/>
-            </visual>
-            <collision>
-                <origin xyz="0 0 0" rpy="0 0 0"/>
-                <geometry>
-                    <mesh filename="package://arm_description/meshes/collision/link_3.stl"/>
-                </geometry>
-            </collision>
-            <inertial>
-                    <origin xyz="0 0 0" rpy="0 0 0"/>
-                    <mass value="4.62"/>
-                    <inertia
-                            ixx="4.37" ixy="-0.00000359" ixz="-0.186"
-                            iyy="4.38" iyz="-0.000112"
-                            izz="0.0236"/>
-            </inertial>
+        <visual>
+            <origin xyz="0 0 0" rpy="0 0 0" />
+            <geometry>
+                <mesh filename="package://arm_description/meshes/visual/link_3.stl" />
+            </geometry>
+            <xacro:material_moving_parts />
+        </visual>
+        <collision>
+            <origin xyz="0 0 0" rpy="0 0 0" />
+            <geometry>
+                <mesh filename="package://arm_description/meshes/collision/link_3.stl" />
+            </geometry>
+        </collision>
+        <inertial>
+            <origin xyz="0 0 0" rpy="0 0 0" />
+            <mass value="4.62" />
+            <inertia ixx="4.37" ixy="-0.00000359" ixz="-0.186" iyy="4.38" iyz="-0.000112" izz="0.0236" />
+        </inertial>
     </link>
     <joint name="q3" type="revolute">
-        <origin xyz="0.560 0 0" rpy="0 0 0"/>
-        <parent link="link_2"/>
-        <child link="link_3"/>
-        <axis xyz="0 1 0"/>
-        <limit effort="100" lower="${-DEG2RAD * 120}" upper="${DEG2RAD * 156}" velocity="${DEG2RAD * 225}"/>
-	<dynamics damping="0.0" friction="0.0"/>
-    </joint>
-	<transmission name="tran3">
+        <origin xyz="0.560 0 0" rpy="0 0 0" />
+        <parent link="link_2" />
+        <child link="link_3" />
+        <axis xyz="0 1 0" />
+        <limit effort="100" lower="${-DEG2RAD * 120}" upper="${DEG2RAD * 156}" velocity="${DEG2RAD * 225}" />
+        <dynamics damping="0.0" friction="0.0" />
+    </joint>
+    <transmission name="tran3">
         <type>transmission_interface/SimpleTransmission</type>
         <joint name="q3">
@@ -156,33 +144,30 @@
     </transmission>
     <link name="link_4">
-            <visual>
-                <origin xyz="0 0 0" rpy="0 0 0"/>
-                <geometry>
-                    <mesh filename="package://arm_description/meshes/visual/link_4.stl"/>
-                </geometry>
-                <xacro:material_moving_parts/>
-            </visual>
-            <collision>
-                <origin xyz="0 0 0" rpy="0 0 0"/>
-                <geometry>
-                    <mesh filename="package://arm_description/meshes/collision/link_4.stl"/>
-                </geometry>
-            </collision>
-            <inertial>
-                    <origin xyz="0 0 0" rpy="0 0 0"/>
-                    <mass value="6.47"/>
-                    <inertia
-                            ixx="6.42" ixy="0.00101" ixz="-2.11"
-                            iyy="7.18" iyz="0.00229"
-                            izz="0.774"/>
-            </inertial>
+        <visual>
+            <origin xyz="0 0 0" rpy="0 0 0" />
+            <geometry>
+                <mesh filename="package://arm_description/meshes/visual/link_4.stl" />
+            </geometry>
+            <xacro:material_moving_parts />
+        </visual>
+        <collision>
+            <origin xyz="0 0 0" rpy="0 0 0" />
+            <geometry>
+                <mesh filename="package://arm_description/meshes/collision/link_4.stl" />
+            </geometry>
+        </collision>
+        <inertial>
+            <origin xyz="0 0 0" rpy="0 0 0" />
+            <mass value="6.47" />
+            <inertia ixx="6.42" ixy="0.00101" ixz="-2.11" iyy="7.18" iyz="0.00229" izz="0.774" />
+        </inertial>
     </link>
     <joint name="q4" type="revolute">
-        <origin xyz="0 0 0.035" rpy="0 0 0"/>
-        <parent link="link_3"/>
-        <child link="link_4"/>
-        <axis xyz="-1 0 0"/>
-        <limit effort="100" lower="${-DEG2RAD * 185}" upper="${DEG2RAD * 185}" velocity="${DEG2RAD * 381}"/>
-	<dynamics damping="0.0" friction="0.0"/>
+        <origin xyz="0 0 0.035" rpy="0 0 0" />
+        <parent link="link_3" />
+        <child link="link_4" />
+        <axis xyz="-1 0 0" />
+        <limit effort="100" lower="${-DEG2RAD * 185}" upper="${DEG2RAD * 185}" velocity="${DEG2RAD * 381}" />
+        <dynamics damping="0.0" friction="0.0" />
     </joint>
     <transmission name="tran4">
@@ -195,35 +180,32 @@
             <mechanicalReduction>1</mechanicalReduction>
         </actuator>
-	</transmission>
+    </transmission>
     <link name="link_5">
-            <visual>
-                <origin xyz="0 0 0" rpy="0 0 0"/>
-                <geometry>
-                    <mesh filename="package://arm_description/meshes/visual/link_5.stl"/>
-                </geometry>
-                <xacro:material_moving_parts/>
-            </visual>
-            <collision>
-                <origin xyz="0 0 0" rpy="0 0 0"/>
-                <geometry>
-                    <mesh filename="package://arm_description/meshes/collision/link_5.stl"/>
-                </geometry>
-            </collision>
-            <inertial>
-                    <origin xyz="0 0 0" rpy="0 0 0"/>
-                    <mass value="0.711"/>
-                    <inertia
-                            ixx="0.704" ixy="-0.000729" ixz="-0.393"
-                            iyy="0.924" iyz="-0.00135"
-                            izz="0.221"/>
-            </inertial>
+        <visual>
+            <origin xyz="0 0 0" rpy="0 0 0" />
+            <geometry>
+                <mesh filename="package://arm_description/meshes/visual/link_5.stl" />
+            </geometry>
+            <xacro:material_moving_parts />
+        </visual>
+        <collision>
+            <origin xyz="0 0 0" rpy="0 0 0" />
+            <geometry>
+                <mesh filename="package://arm_description/meshes/collision/link_5.stl" />
+            </geometry>
+        </collision>
+        <inertial>
+            <origin xyz="0 0 0" rpy="0 0 0" />
+            <mass value="0.711" />
+            <inertia ixx="0.704" ixy="-0.000729" ixz="-0.393" iyy="0.924" iyz="-0.00135" izz="0.221" />
+        </inertial>
     </link>
     <joint name="q5" type="revolute">
-        <origin xyz="0.515 0 0" rpy="0 0 0"/>
-        <parent link="link_4"/>
-        <child link="link_5"/>
-        <axis xyz="0 1 0"/>
-        <limit effort="100" lower="${-DEG2RAD * 120}" upper="${DEG2RAD * 120}" velocity="${DEG2RAD * 311}"/>
-	<dynamics damping="0.0" friction="0.0"/>
+        <origin xyz="0.515 0 0" rpy="0 0 0" />
+        <parent link="link_4" />
+        <child link="link_5" />
+        <axis xyz="0 1 0" />
+        <limit effort="100" lower="${-DEG2RAD * 120}" upper="${DEG2RAD * 120}" velocity="${DEG2RAD * 311}" />
+        <dynamics damping="0.0" friction="0.0" />
     </joint>
     <transmission name="tran5">
@@ -238,33 +220,30 @@
     </transmission>
     <link name="link_6">
-            <visual>
-                <origin xyz="0 0 0" rpy="0 0 0"/>
-                <geometry>
-                    <mesh filename="package://arm_description/meshes/visual/link_6.stl"/>
-                </geometry>
-                <xacro:material_moving_parts/>
-            </visual>
-            <collision>
-                <origin xyz="0 0 0" rpy="0 0 0"/>
-                <geometry>
-                    <mesh filename="package://arm_description/meshes/collision/link_6.stl"/>
-                </geometry>
-            </collision>
-            <inertial>
-                    <origin xyz="0 0 0" rpy="0 0 0"/>
-                    <mass value="0.0225"/>
-                    <inertia
-                            ixx="0.0223" ixy="0.0" ixz="-0.0137"
-                            iyy="0.0307" iyz="0.0"
-                            izz="0.00844"/>
-            </inertial>
+        <visual>
+            <origin xyz="0 0 0" rpy="0 0 0" />
+            <geometry>
+                <mesh filename="package://arm_description/meshes/visual/link_6.stl" />
+            </geometry>
+            <xacro:material_moving_parts />
+        </visual>
+        <collision>
+            <origin xyz="0 0 0" rpy="0 0 0" />
+            <geometry>
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
File: arm_description/urdf/colors.xacro (robot description, xacro)
@@ -3,8 +3,8 @@
   <!-- default colors for robots -->
   <!-- RAL 9016: base frame (traffic white) -->
-  <xacro:property name="color_base_frame" value="${241/255} ${240/255} ${234/255} 1.0"/>
+  <xacro:property name="color_base_frame" value="${241/255} ${240/255} ${234/255} 1.0" />
   <!-- RAL 9016: moving parts (traffic white) -->
-  <xacro:property name="color_moving_parts" value="${241/255} ${240/255} ${234/255} 1.0"/>
+  <xacro:property name="color_moving_parts" value="${241/255} ${240/255} ${234/255} 1.0" />
   <!-- RAL 9016: moving parts (traffic white) -->
-  <xacro:property name="color_sensors" value="${255/255} ${17/255} ${0/255} 1.0"/>
+  <xacro:property name="color_sensors" value="${255/255} ${17/255} ${0/255} 1.0" />
 </robot>

File: arm_description/urdf/constants.xacro (robot description, xacro)
@@ -1,3 +1,3 @@
-<?xml version="1.0"?>
+<?xml version="1.0" ?>
 <robot xmlns:xacro="http://wiki.ros.org/xacro">
   <xacro:property name="DEG2RAD" value="0.017453292519943295" />

File: arm_description/urdf/materials.xacro (robot description, xacro)
@@ -1,18 +1,18 @@
-<?xml version="1.0"?>
+<?xml version="1.0" ?>
 <robot xmlns:xacro="http://wiki.ros.org/xacro">
-  <xacro:include filename="$(find arm_description)/urdf/colors.xacro"/>
+  <xacro:include filename="$(find arm_description)/urdf/colors.xacro" />
   <xacro:macro name="material_base_frame">
     <material name="">
-      <color rgba="${color_base_frame}"/>
+      <color rgba="${color_base_frame}" />
     </material>
   </xacro:macro>
   <xacro:macro name="material_moving_parts">
     <material name="">
-      <color rgba="${color_moving_parts}"/>
+      <color rgba="${color_moving_parts}" />
     </material>
   </xacro:macro>
   <xacro:macro name="material_sensors">
     <material name="">
-      <color rgba="${color_sensors}"/>
+      <color rgba="${color_sensors}" />
     </material>
   </xacro:macro>

Commit message: Splitted the urdf. For now camera located in the separate xacro file

File: arm_description/urdf/arm.urdf.xacro (robot description, xacro)
@@ -3,4 +3,8 @@
     <xacro:include filename="$(find arm_description)/urdf/constants.xacro" />
     <xacro:include filename="$(find arm_description)/urdf/materials.xacro" />
+    <xacro:arg name="with_camera" default="false" />
+    <xacro:if value="$(arg with_camera)">
+        <xacro:include filename="$(find arm_description)/urdf/camera.xacro" />
+    </xacro:if>
     <link name="world" />
     <link name="base_link">
@@ -263,68 +267,4 @@
         <origin xyz="0 0 0" rpy="0 ${DEG2RAD * 90} 0" />
     </joint>
-    <!-- Camera -->
-    <link name="link_camera">
-        <visual>
-            <origin xyz="0 0 0" rpy="0 0 0" />
-            <geometry>
-                <box size="0.05 0.05 0.05" />
-            </geometry>
-            <xacro:material_sensors />
-        </visual>
-        <collision>
-            <origin xyz="0 0 0" rpy="0 0 0" />
-            <geometry>
-                <box size="0.05 0.05 0.05" />
-            </geometry>
-        </collision>
-        <inertial>
-            <origin xyz="0 0 0" rpy="0 0 0" />
-            <mass value="1e-5" />
-            <inertia ixx="1e-6" ixy="0.0" ixz="0.0" iyy="1e-6" iyz="0.0" izz="1e-6" />
-        </inertial>
-    </link>
-    <joint name="joint_camera" type="fixed">
-        <axis xyz="0 1 0" />
-        <origin xyz="0.1 0 0.1" rpy="0 0 0" />
-        <parent link="link_2" />
-        <child link="link_camera" />
-    </joint>
-    <!-- Camera -->
-    <gazebo reference="link_camera">
-        <sensor type="camera" name="camera">
-            <update_rate>30.0</update_rate>
-            <camera name="head">
-                <horizontal_fov>1.3962634</horizontal_fov>
-                <image>
-                    <width>800</width>
-                    <height>800</height>
-                    <format>R8G8B8</format>
-                </image>
-                <clip>
-                    <near>0.02</near>
-                    <far>300</far>
-                </clip>
-                <noise>
-                    <type>gaussian</type>
-                    <mean>0.0</mean>
-                    <stddev>0.007</stddev>
-                </noise>
-            </camera>
-            <plugin name="camera_controller" filename="libgazebo_ros_camera.so">
-                <alwaysOn>true</alwaysOn>
-                <updateRate>0.0</updateRate>
-                <cameraName>/kuka_arm/camera</cameraName>
-                <imageTopicName>image_raw</imageTopicName>
-                <cameraInfoTopicName>camera_info</cameraInfoTopicName>
-                <frameName>link_camera</frameName>
-                <hackBaseline>0.07</hackBaseline>
-                <distortionK1>0.0</distortionK1>
-                <distortionK2>0.0</distortionK2>
-                <distortionK3>0.0</distortionK3>
-                <distortionT1>0.0</distortionT1>
-                <distortionT2>0.0</distortionT2>
-            </plugin>
-        </sensor>
-    </gazebo>
     <!-- Controllers -->
     <gazebo>
